File: can.kicad_sch (KiCad schematic)
At the start: 5 parts, among them J1 Conn_01x02, U2 TJA1051T

Commit message: deployment release
Parts:
- removed JP1: SolderJumper_2_Bridged, Jumper:SolderJumper-2_P1.3mm_Bridged_Pad1.0x1.5mm, symbol Jumper:SolderJumper_2_Bridged
- added JP3: Jumper_2_Bridged, Connector_PinHeader_2.00mm:PinHeader_1x02_P2.00mm_Vertical, symbol Jumper:Jumper_2_Bridged
Connections:
- net at J1.1 (Pin_1), U2.6 (CANL): now also JP3.2 (B)
- net at R2.2: now also JP3.1 (A)
Changed lines of the file:
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@@
 (kicad_sch (version 20230121) (generator eeschema)
   (paper "A4")
-  (junction (at 93.98 81.28) (diameter 0) (color 0 0 0 0)
-  )
   (junction (at 93.98 95.25) (diameter 0) (color 0 0 0 0)
   )
+  (junction (at 93.98 78.74) (diameter 0) (color 0 0 0 0)
+  )
   (wire (pts (xy 93.98 95.25) (xy 111.76 95.25))
     (stroke (width 0) (type default))
@@
     (stroke (width 0) (type default))
   )
-  (wire (pts (xy 73.66 86.36) (xy 73.66 81.28))
+  (wire (pts (xy 73.66 86.36) (xy 73.66 78.74))
     (stroke (width 0) (type default))
   )
@@
     (stroke (width 0) (type default))
   )
-  (wire (pts (xy 73.66 81.28) (xy 93.98 81.28))
-    (stroke (width 0) (type default))
-  )
   (wire (pts (xy 139.7 86.36) (xy 152.4 86.36))
     (stroke (width 0) (type default))
   )
-  (wire (pts (xy 93.98 81.28) (xy 114.3 81.28))
+  (wire (pts (xy 73.66 78.74) (xy 93.98 78.74))
+    (stroke (width 0) (type default))
+  )
+  (wire (pts (xy 114.3 78.74) (xy 114.3 81.28))
+    (stroke (width 0) (type default))
+  )
+  (wire (pts (xy 93.98 78.74) (xy 114.3 78.74))
     (stroke (width 0) (type default))
   )
@@
     )
   )
+  (symbol (lib_id "Jumper:Jumper_2_Bridged") (at 93.98 83.82 90) (unit 1)
+    (in_bom yes) (on_board yes) (dnp no) (fields_autoplaced)
+    (property "Reference" "JP3" (at 95.25 82.55 90)
+      (effects (font (size 1.27 1.27)) (justify right))
+    )
+    (property "Value" "Jumper_2_Bridged" (at 95.25 85.09 90)
+      (effects (font (size 1.27 1.27)) (justify right))
+    )
+    (property "Footprint" "Connector_PinHeader_2.00mm:PinHeader_1x02_P2.00mm_Vertical" (at 93.98 83.82 0)
+      (effects (font (size 1.27 1.27)) hide)
+    )
+    (property "Datasheet" "~" (at 93.98 83.82 0)
+      (effects (font (size 1.27 1.27)) hide)
+    )
+    (pin "2")
+    (pin "1")
+    (instances
+      (project "cyberboard"
+        (path "/69441227-0733-4ee0-b881-4d19bfeb4a0a/936da2af-c82b-43b6-be61-521cfea06692"
+          (reference "JP3") (unit 1)
+        )
+      )
+    )
+  )
   (symbol (lib_id "power:GND") (at 127 73.66 180) (unit 1)
     (in_bom yes) (on_board yes) (dnp no) (fields_autoplaced)
@@
         )
       )
-    )
-  )
-  (symbol (lib_id "Jumper:SolderJumper_2_Bridged") (at 93.98 85.09 90) (unit 1)
-    (in_bom yes) (on_board yes) (dnp no) (fields_autoplaced)
-    (property "Reference" "JP1" (at 96.52 84.455 90)
-      (effects (font (size 1.27 1.27)) (justify right))
-    )
-    (property "Value" "SolderJumper_2_Bridged" (at 96.52 86.995 90)
-      (effects (font (size 1.27 1.27)) (justify right))
-    )
-    (property "Footprint" "Jumper:SolderJumper-2_P1.3mm_Bridged_Pad1.0x1.5mm" (at 93.98 85.09 0)
-      (effects (font (size 1.27 1.27)) hide)
-    )
-    (property "Datasheet" "~" (at 93.98 85.09 0)
-      (effects (font (size 1.27 1.27)) hide)
-    )
-    (pin "1")
-    (pin "2")
-    (instances
-      (project "cyberboard"
-        (path "/69441227-0733-4ee0-b881-4d19bfeb4a0a/936da2af-c82b-43b6-be61-521cfea06692"
-          (reference "JP1") (unit 1)
-        )
-      )
