File: cyberboard.kicad_sch (KiCad schematic)
At the start: 13 parts, among them U6 ESP32-S3-WROOM-1

Commit message: deployment release
Parts:
- added J4, J8: Conn_01x14, Connector_PinSocket_2.54mm:PinSocket_1x14_P2.54mm_Vertical, symbol Connector_Generic:Conn_01x14
Connections:
- net GPIO0_1 is gone; now on net I2C_SCL: U6.23 (GPIO21)
- net GPIO0_2 is gone; now on net I2C_SDA: U6.24 (GPIO47/SPICLK_P/SUBSPICLK_P_DIFF)
- net +3.3V: now also J4.1 (3.3V), J8.1 (3.3V)
- net CAN_RX: now also U6.21 (GPIO13/TOUCH13/ADC2_CH2/FSPIQ/FSPIIO7/SUBSPIQ); no longer U6.6 (GPIO6/TOUCH6/ADC1_CH5)
- net CAN_TX: now also U6.22 (GPIO14/TOUCH14/ADC2_CH3/FSPIWP/FSPIDQS/SUBSPIWP); no longer U6.5 (GPIO5/TOUCH5/ADC1_CH4)
- net GND: now also J4.13 (GND), J4.2 (GND), J8.13 (GND), J8.2 (GND)
- net GPIO1_1: now also U6.6 (GPIO6/TOUCH6/ADC1_CH5), J8.3 (GPIO1); no longer U6.7 (GPIO7/TOUCH7/ADC1_CH6)
- net GPIO1_2: now also U6.7 (GPIO7/TOUCH7/ADC1_CH6), J8.4 (GPIO2); no longer U6.8 (GPIO15/U0RTS/ADC2_CH4/XTAL_32K_P)
- net GPIO1_3: now also U6.8 (GPIO15/U0RTS/ADC2_CH4/XTAL_32K_P), J8.5 (GPIO3); no longer U6.9 (GPIO16/U0CTS/ADC2_CH5/XTAL_32K_N)
- net GPIO1_4: now also U6.9 (GPIO16/U0CTS/ADC2_CH5/XTAL_32K_N), J8.6 (GPIO4); no longer U6.10 (GPIO17/U1TXD/ADC2_CH6)
- net GPIO2_1: now also U6.37 (U0TXD/GPIO43/CLK_OUT1), J4.3 (GPIO1); no longer U6.35 (MTMS/GPIO42)
- net GPIO2_2: now also U6.36 (U0RXD/GPIO44/CLK_OUT2), J4.4 (GPIO2); no longer U6.34 (MTDI/GPIO41/CLK_OUT1)
- net GPIO2_3: now also U6.35 (MTMS/GPIO42), J4.5 (GPIO3); no longer U6.33 (MTDO/GPIO40/CLK_OUT2)
- net GPIO2_4: now also U6.34 (MTDI/GPIO41/CLK_OUT1), J4.6 (GPIO4); no longer U6.32 (MTCK/GPIO39/CLK_OUT3/SUBSPICS1)
- net GPIO_ACTION: now also U6.38 (GPIO2/TOUCH2/ADC1_CH1); no longer U6.31 (GPIO38/FSPIWP/SUBSPIWP)
- net GPIO_LED: now also U6.39 (GPIO1/TOUCH1/ADC1_CH0); no longer U6.30 (SPIDQS/GPIO37/FSPIQ/SUBSPIQ)
- net I2C_SCL: no longer U6.11 (GPIO18/U1RXD/ADC2_CH7/CLK_OUT3)
- net I2C_SDA: no longer U6.12 (GPIO8/TOUCH8/ADC1_CH7/SUBSPICS1)
- net IMU_CS: now also U6.11 (GPIO18/U1RXD/ADC2_CH7/CLK_OUT3); no longer U6.37 (U0TXD/GPIO43/CLK_OUT1)
- net IMU_INT: now also U6.4 (GPIO4/TOUCH4/ADC1_CH3); no longer U6.39 (GPIO1/TOUCH1/ADC1_CH0)
- net IMU_SCL: now also U6.15 (GPIO3/TOUCH3/ADC1_CH2); no longer U6.36 (U0RXD/GPIO44/CLK_OUT2)
- net IMU_SDA: now also U6.16 (GPIO46); no longer U6.4 (GPIO4/TOUCH4/ADC1_CH3)
- net IMU_SDO: now also U6.5 (GPIO5/TOUCH5/ADC1_CH4); no longer U6.38 (GPIO2/TOUCH2/ADC1_CH1)
- net GPIO1_7: now reaches U6.17 (GPIO9/TOUCH9/ADC1_CH8/FSPIHD/SUBSPIHD)
- net GPIO1_7: now also J8.9 (GPIO7)
- net GPIO1_8: now reaches U6.18 (GPIO10/TOUCH10/ADC1_CH9/FSPICS0/FSPIIO4/SUBSPICS0)
- net GPIO1_8: now also J8.10 (GPIO8)
- net GPIO1_9: now reaches U6.19 (GPIO11/TOUCH11/ADC2_CH0/FSPID/FSPIIO5/SUBSPID)
- net GPIO1_9: now also J8.11 (GPIO9)
- net GPIO1_10: now reaches U6.20 (GPIO12/TOUCH12/ADC2_CH1/FSPICLK/FSPIIO6/SUBSPICLK)
- net GPIO1_10: now also J8.12 (GPIO10)
- net GPIO2_10: now reaches U6.28 (SPIIO6/GPIO35/FSPID/SUBSPID)
- net GPIO2_10: now also J4.12 (GPIO10)
- net GPIO2_9: now reaches U6.29 (SPIIO7/GPIO36/FSPICLK/SUBSPICLK)
- net GPIO2_9: now also J4.11 (GPIO9)
- net GPIO0_3: no longer names the net of U6.25 (GPIO48/SPICLK_N/SUBSPICLK_N_DIFF)
- net GPIO0_4: no longer names the net of U6.26 (GPIO45)
- new net +5V: J4.14 (5V), J8.14 (5V)
- new net GPIO1_5: J8.7 (GPIO5), U6.10 (GPIO17/U1TXD/ADC2_CH6)
- new net GPIO1_6: J8.8 (GPIO6), U6.12 (GPIO8/TOUCH8/ADC1_CH7/SUBSPICS1)
- new net GPIO2_5: J4.7 (GPIO5), U6.33 (MTDO/GPIO40/CLK_OUT2)
- new net GPIO2_6: J4.8 (GPIO6), U6.32 (MTCK/GPIO39/CLK_OUT3/SUBSPICS1)
- new net GPIO2_7: J4.9 (GPIO7), U6.31 (GPIO38/FSPIWP/SUBSPIWP)
- new net GPIO2_8: J4.10 (GPIO8), U6.30 (SPIDQS/GPIO37/FSPIQ/SUBSPIQ)
- no-connect marks 11 -> 3
Other:
- removed sheet GPIO
- removed sheet GPIO1
- removed sheet GPIO2
