File: gpio.kicad_sch (KiCad schematic)
At the start: 1 part, among them J4 Conn_01x07

Commit message: deployment release
Parts:
- J4: value Conn_01x07 -> Conn_01x12
Changed lines of the file:
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@@
       (effects (font (size 1.27 1.27)) (justify left))
     )
-    (property "Value" "Conn_01x07" (at 106.68 68.58 0)
+    (property "Value" "Conn_01x12" (at 106.68 68.58 0)
       (effects (font (size 1.27 1.27)) (justify left))
     )
