File: power.kicad_sch (KiCad schematic)
At the start: 15 parts, among them J2 USB_C_Receptacle_USB2.0, J3 5024940670, U3 D3V3XA4B10LP, U4 TLV75801PDRV

Commit message: deployment release
Parts:
- removed JP2: SolderJumper_3_Bridged12, Jumper:SolderJumper-3_P1.3mm_Bridged12_RoundedPad1.0x1.5mm_NumberLabels, symbol Jumper:SolderJumper_3_Bridged12
- removed R6: 1M, Resistor_SMD:R_0805_2012Metric, symbol Device:R_Small
- removed R7: 200k, Resistor_SMD:R_0805_2012Metric, symbol Device:R_Small
- removed U4: TLV75801PDRV, Package_SON:WSON-6-1EP_2x2mm_P0.65mm_EP1x1.6mm, symbol Regulator_Linear:TLV75801PDRV
- added JP1: Jumper_3_Bridged12, Connector_PinHeader_2.00mm:PinHeader_1x03_P2.00mm_Vertical, symbol Jumper:Jumper_3_Bridged12
- added U1: AMS1117-3.3, Package_TO_SOT_SMD:SOT-223-3_TabPin2, symbol Regulator_Linear:AMS1117-3.3
Connections:
- net +3.3V: now also U1.2 (VO)
- net +5V: now also JP1.2 (C), U1.3 (VI)
- net 5V_PDB: now also JP1.1 (A)
- net 5V_USB: now also JP1.3 (B)
- net GND: now also U1.1 (GND)
Other:
- moved on the sheet: C3, C4, D2, R8
